Commit message: Update urdf.xacro box_bot file to have correct intertial properties and change size of wheels

File: box_bot_sim/urdf/box_bot.urdf.xacro (robot description, xacro)
@@ -1,9 +1,10 @@
 <?xml version="1.0"?>
 <robot name="box_bot" xmlns:xacro="http://www.ros.org/wiki/xacro">
+<xacro:include filename="inertial_macros.xacro"/>
   <link name="base_link"/>
   <joint name="chassis_joint" type="fixed">
     <parent link="base_link"/>
     <child link="chassis"/>
-    <origin xyz="0 0 0.1"/>
+    <origin xyz="0 0 0" rpy="0 0 0"/>
   </joint>
   <link name="chassis">
@@ -15,21 +16,19 @@
       <geometry><box size="0.4 0.3 0.15"/></geometry>
     </collision>
-    <inertial>
-      <mass value="1.0"/>
-      <inertia ixx="0.01" ixy="0" ixz="0" iyy="0.01" iyz="0" izz="0.01"/>
-    </inertial>
+    <xacro:inertial_box mass="1.0" x="0.4" y="0.3" z="0.15">
+      <origin xyz="0 0 0" rpy="0 0 0"/>
+    </xacro:inertial_box>
   </link>
   <link name="left_wheel">
     <visual>
-      <geometry><cylinder radius="0.1" length="0.04"/></geometry>
+      <geometry><cylinder radius="0.05" length="0.04"/></geometry>
       <material name="black"><color rgba="0 0 0 1"/></material>
     </visual>
     <collision>
-      <geometry><cylinder radius="0.1" length="0.04"/></geometry>
+      <geometry><cylinder radius="0.05" length="0.04"/></geometry>
     </collision>
-    <inertial>
-      <mass value="0.1"/>
-      <inertia ixx="0.001" ixy="0" ixz="0" iyy="0.001" iyz="0" izz="0.001"/>
-    </inertial>
+    <xacro:inertial_cylinder mass="0.1" length="0.04" radius="0.05">
+      <origin xyz="0 0 0" rpy="0 0 0"/>
+    </xacro:inertial_cylinder>
   </link>
   <joint name="left_wheel_joint" type="continuous">
@@ -41,14 +40,13 @@
   <link name="right_wheel">
     <visual>
-      <geometry><cylinder radius="0.1" length="0.04"/></geometry>
+      <geometry><cylinder radius="0.05" length="0.04"/></geometry>
       <material name="black"><color rgba="0 0 0 1"/></material>
     </visual>
     <collision>
-      <geometry><cylinder radius="0.1" length="0.04"/></geometry>
+      <geometry><cylinder radius="0.05" length="0.04"/></geometry>
     </collision>
-    <inertial>
-      <mass value="0.1"/>
-      <inertia ixx="0.001" ixy="0" ixz="0" iyy="0.001" iyz="0" izz="0.001"/>
-    </inertial>
+    <xacro:inertial_cylinder mass="0.1" length="0.04" radius="0.05">
+      <origin xyz="0 0 0" rpy="0 0 0"/>
+    </xacro:inertial_cylinder>
   </link>
   <joint name="right_wheel_joint" type="continuous">
@@ -56,5 +54,5 @@
     <child link="right_wheel"/>
     <origin xyz="0 -0.175 -0.05" rpy="1.5708 0 0"/>
-    <axis xyz="0 0 1"/>
+    <axis xyz="0 0 -1"/>
   </joint>
   <link name="caster">
@@ -65,13 +63,12 @@
       <geometry><sphere radius="0.05"/></geometry>
     </collision>
-    <inertial>
-      <mass value="0.1"/>
-      <inertia ixx="0.0001" ixy="0" ixz="0" iyy="0.0001" iyz="0" izz="0.0001"/>
-    </inertial>
+    <xacro:inertial_sphere mass="0.1" radius="0.05">
+      <origin xyz="0 0 0" rpy="0 0 0"/>
+    </xacro:inertial_sphere>
   </link>
   <joint name="caster_joint" type="fixed">
     <parent link="chassis"/>
     <child link="caster"/>
-    <origin xyz="0.15 0 -0.1"/>
+    <origin xyz="0.15 0 -0.05"/>
   </joint>
   <gazebo>
